File: pcb/Diode_keyboard/diode_keyboard.brd (EAGLE design)
At the start: 92.7 x 84.8 mm, 213 parts, among them IC1 74ALS04D, IC2 4051D, IC3 4051D

Commit message: after autorouter
Routing:
- net X1: track 0.00 -> 168.4 mm, vias 0 -> 1
- net X3: track 0.00 -> 142.3 mm, vias 0 -> 1
- net X0: track 0.00 -> 141.7 mm, vias 0 -> 2
- net X6: track 0.00 -> 130.4 mm, vias 0 -> 2
- net X4: track 0.00 -> 127.8 mm, vias 0 -> 2
- net X2: track 0.00 -> 126.2 mm, vias 0 -> 2
- net X5: track 0.00 -> 118.4 mm, vias 0 -> 1
- net C: track 0.00 -> 117.0 mm, vias 0 -> 1
- net +3V3: track 0.00 -> 115.4 mm, vias 0 -> 2
- net Y7: track 0.00 -> 110.6 mm
- net Y6: track 0.00 -> 109.1 mm, vias 0 -> 1
- net Y4: track 0.00 -> 106.6 mm
- net GND: track 0.00 -> 104.3 mm, vias 0 -> 3
- net X7: track 0.00 -> 103.1 mm, vias 0 -> 3
- net Y5: track 0.00 -> 97.5 mm
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